File: UKHASnet wifi pcb/UKHASnetWifiNode.sch (EAGLE design)
At the start: 24 parts, among them U1 ATMEGA328P-AU, U2 LM2937IMP-5.0

Commit message: Schematic tidied
Parts:
- C1, C6: value (none) -> 100nf
- C2: value 0.1uf -> 100nf
Other:
- note added: "Please set ADC resistor dividers depending on input voltage range."
- note added: "RFM69HW"
- moved on the sheet: ADC, C1, C2, C5, C6, GPIO, ICSP1, JP1, JP2, R4, R5, R6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
